Commit message: Stop tracking turtlebot folder

File: mycobot_ros/mycobot_description/urdf/mycobot_320_m5_2022/new_mycobot_pro_320_m5_2022_gripper.urdf (robot description, URDF)
Before this commit: robot firefighter, 20 links, 19 joints
Links:
- removed link wall_link
- added link wall_link1; collision box size=0.05 1.2 0.8; visual box size=0.05 1.2 0.8
- added link wall_link2; collision box size=1.15 0.05 0.8; visual box size=1.15 0.05 0.8
- link base: geometry collision cylinder length=0.096 radius=0.05; visual mesh filename=package://mycobot_description/urdf/mycobot_320_m5_2022/base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
- link camlink: geometry collision box size=0.05 0.045 0.01; visual mesh filename=package://mycobot_description/urdf/mycobot_320_m5_2022/came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
- link link1: geometry collision cylinder length=0.114 radius=0.025; visual mesh filename=package://mycobot_description/urdf/mycobot_320_m5_2022/link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
- link link2: geometry collision cylinder length=0.203 radius=0.025; visual mesh filename=package://mycobot_description/urdf/mycobot_320_m5_2022/link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
- link link3: geometry collision cylinder length=0.18 radius=0.025; visual mesh filename=package://mycobot_description/urdf/mycobot_320_m5_2022/link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
- link link4: geometry collision cylinder length=0.073 radius=0.02; visual mesh filename=package://mycobot_description/urdf/mycobot_320_m5_2022/link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
- link link5: geometry collision cylinder length=0.078 radius=0.025; visual mesh filename=package://mycobot_description/urdf/mycobot_320_m5_2022/link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
- link link6: geometry collision cylinder length=0.0225 radius=0.02; visual mesh filename=package://mycobot_description/urdf/mycobot_320_m5_2022/link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
Joints:
- removed joint wall_joint
- added joint wall_joint1: type fixed, parent base, child wall_link1, origin xyz=0 0 0 rpy=0 0 0 
- added joint wall_joint2: type fixed, parent base, child wall_link2, origin xyz=0 0 0 rpy=0 0 0 

Commit message: Upgate06-12

File: mycobot_ros/mycobot_description/urdf/mycobot_320_m5_2022/new_mycobot_pro_320_m5_2022_gripper.urdf (robot description, URDF)
Before this commit: robot firefighter, 21 links, 20 joints
Links:
- added link table_link; collision box size=0.4 0.7 0.05; collision box size=0.7 0.4 0.05
Joints:
- added joint table_to_base: type fixed, parent base, child table_link, origin xyz=-0.485 -0.05 -0.05 rpy=0 0 3.14159
